File: KiCAD/ZorroRAM.kicad_pcb (KiCad board)
At the start: 2 copper layers, 172.3 x 85.3 mm, 20 parts, among them J1 Xilinx Program Header, U2 AP2210N-3.3TRG1, U3 74LVC245, U4 74LVC245, U5 XC9572XL-10VQ64C, U6 K4E641612D

Commit message: Add files via upload
Parts:
- removed C3: 0.1uF, Capacitor_SMD:C_1206_3216Metric
- J1: value Xilinx Program Header -> Conn_01x06_Male
Connections:
- ZorroSlot1 pad 1: GND -> Net-(ZorroSlot1-Pad1)
- ZorroSlot1 pad 3: GND -> Net-(ZorroSlot1-Pad3)
- ZorroSlot1 pad 99: GND -> Net-(ZorroSlot1-Pad99)
Routing:
- net /READ: track 83.1 -> 115.9 mm, vias 3 -> 5
Other:
- board text added: "XILINX Program Header"
- board text added: "ZoRAM Amiga 2000 8 Megabyte Fast Ram Expansion v 0.6 jasonsbeer https://github.com/jasonsbeer/ZoRAM-Amiga-2000-RAM Only AMIGA makes it possible."
- board text removed: "ZoRAM 8 Megabyte Fast Ram Expansion Amiga 2000 v 0.5 jasonsbeer Only AMIGA makes it possible."
