File: KiCAD/ZorroRAM.sch (KiCad schematic (older format))
At the start: 19 parts, among them J1 Conn_01x06_Male, U2 AP2210N-3.3TRG1, U3 74LVC245, U4 74LVC245, U5 XC9572XL-10VQ64C, U6 K4E641612D

Commit message: Add files via upload
Parts:
- ZorroSlot1: symbol Amiga-Library:ZorroCardEdge -> ZorroRAM-rescue:ZorroCardEdge-Amiga-Library
Connections:
- net GND: no longer ZorroSlot1.1 (Pin_1), ZorroSlot1.3 (Pin_3), ZorroSlot1.99 (Pin99)
Changed lines of the file:
@@
 $EndDescr
 $Comp
-L Amiga-Library:ZorroCardEdge ZorroSlot1
+L ZorroRAM-rescue:ZorroCardEdge-Amiga-Library ZorroSlot1
 U 1 1 60310C7A
 P 1400 3450
@@
 F 3 "" H 8200 1600 50  0001 C CNN
 	1    8200 1600
-	1    0    0    -1
-$EndComp
-Wire Wire Line
-	1200 1750 1200 1650
-Wire Wire Line
-	1200 1650 800  1650
-Wire Wire Line
-	800  1650 800  1700
-Connection ~ 1200 1650
-$Comp
-L power:GND #PWR0110
-U 1 1 60362CA3
-P 800 1700
-F 0 "#PWR0110" H 800 1450 50  0001 C CNN
-F 1 "GND" H 805 1527 50  0000 C CNN
-F 2 "" H 800 1700 50  0001 C CNN
-F 3 "" H 800 1700 50  0001 C CNN
-	1    800  1700
 	1    0    0    -1
 $EndComp
@@
 BA23
 Wire Wire Line
-	1200 6550 1200 6750
-Wire Wire Line
-	1200 6750 1450 6750
-Wire Wire Line
 	1700 6750 1700 6550
 $Comp
@@
 	1    0    0    -1
 $EndComp
-Connection ~ 1450 6750
 Wire Wire Line
 	1450 6750 1700 6750
